File: hardware/connectors.kicad_sch (KiCad schematic)
At the start: 17 parts, among them J1 TYPE-C16PIN, J3 PPTC202LFBN-RC, J4 Conn_02x05_Odd_Even, J5 Conn_01x07_Pin, U5 HT42B534-2_C493361, U6 TPD6E004RSER

Commit message: Added schematic title block info, and pdf version of schematic.
Other:
- company: (none) -> Vespid
- title: (none) -> Orbweaver
Changed lines of the file:
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@@
 	(generator_version "9.0")
 	(paper "A4")
+	(title_block
+		(title "Orbweaver")
+		(date "2026-09-28")
+		(rev "1")
+		(company "Vespid")
+		(comment 1 "github.com/vespid-tech/orbweaver")
+		(comment 2 "www.vespidtech.com")
+		(comment 3 "License: CERN-OHL-S-2.0")
+	)
 	(junction
 		(at 52.07 130.81)
