File: hardware/mcu.kicad_sch (KiCad schematic)
At the start: 40 parts, among them U1 CC1310F128RGZR, Y1 TSX-322524.0000MF15X-AC0, Y2 FC-135_32.7680KA-AG3

Commit message: Added schematic title block info, and pdf version of schematic.
Other:
- sheet Memory: file untitled.kicad_sch -> memory.kicad_sch
- company: (none) -> Vespid
- title: Bridge 0 -> Orbweaver
Changed lines of the file:
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@@
 	(paper "B")
 	(title_block
-		(title "Bridge 0")
+		(title "Orbweaver")
+		(date "2026-09-28")
+		(rev "1")
+		(company "Vespid")
+		(comment 1 "github.com/vespid-tech/orbweaver")
+		(comment 2 "www.vespidtech.com")
+		(comment 3 "License: CERN-OHL-S-2.0")
 	)
 	(junction
@@
 		)
 		(instances
-			(project "bridge_0"
+			(project "mcu"
 				(path "/60452dac-b6a4-46ed-b82d-e4d65188999a"
 					(page "4")
@@
 		)
 		(instances
-			(project "bridge_0"
+			(project "mcu"
 				(path "/60452dac-b6a4-46ed-b82d-e4d65188999a"
 					(page "2")
@@
 		)
 		(instances
-			(project "bridge_0"
+			(project "mcu"
 				(path "/60452dac-b6a4-46ed-b82d-e4d65188999a"
 					(page "3")
@@
 			)
 		)
-		(property "Sheetfile" "untitled.kicad_sch"
+		(property "Sheetfile" "memory.kicad_sch"
 			(at 24.13 255.8546 0)
 			(effects
@@
 		)
 		(instances
-			(project "bridge_0"
+			(project "mcu"
 				(path "/60452dac-b6a4-46ed-b82d-e4d65188999a"
 					(page "5")
