File: hardware/power.kicad_sch (KiCad schematic)
At the start: 12 parts, among them U2 XC6206P332MR, U3 TPS2113APW

Commit message: Added schematic title block info, and pdf version of schematic.
Other:
- company: (none) -> Vespid
- title: Bridge_0 -> Orbweaver
Changed lines of the file:
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@@
 	(paper "A4")
 	(title_block
-		(title "Bridge_0")
+		(title "Orbweaver")
+		(date "2026-09-28")
+		(rev "1")
+		(company "Vespid")
+		(comment 1 "github.com/vespid-tech/orbweaver")
+		(comment 2 "www.vespidtech.com")
+		(comment 3 "License: CERN-OHL-S-2.0")
 	)
 	(text "use USB power as long\nas it's above 4.1 VDC.\nOtherwise, use +5 from\nthe Raspberry Pi."
