File: hardware/rf.kicad_sch (KiCad schematic)
At the start: 3 parts, among them J2 RFPC-SMA27-F, U4 LFB18868MBG9E212

Commit message: Added schematic title block info, and pdf version of schematic.
Other:
- company: (none) -> Vespid
- title: (none) -> Orbweaver
Changed lines of the file:
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@@
 	(generator_version "9.0")
 	(paper "A4")
+	(title_block
+		(title "Orbweaver")
+		(date "2026-09-28")
+		(rev "1")
+		(company "Vespid")
+		(comment 1 "github.com/vespid-tech/orbweaver")
+		(comment 2 "www.vespidtech.com")
+		(comment 3 "License: CERN-OHL-S-2.0")
+	)
 	(junction
 		(at 210.82 95.25)
