File: hardware/orbweaver.kicad_pcb (KiCad board)
At the start: 4 copper layers, 56.5 x 65 mm, 86 parts, among them IC1 ZD25WQ80COIGR, J1 TYPE-C16PIN, J2 RFPC-SMA27-F, J3 PPTC202LFBN-RC, J4 Conn_02x05_Odd_Even, J5 Conn_01x07_Pin, J6 DNI, U1 CC1310F128RGZR, U2 XC6206P332MR, U3 TPS2113APW, U4 LFB18868MBG9E212, U5 HT42B534-2_C493361, U6 TPD6E004RSER, U7 CAT24C32WI-GT3, Y1 TSX-322524.0000MF15X-AC0, Y2 FC-135_32.7680KA-AG3

Commit message: Fixed firmware python scripts. Updated public schematics.
Parts:
- added J7: DNI, Connector_PinHeader_2.54mm:PinHeader_1x02_P2.54mm_Vertical, F.Cu at (138.5, 74.5)
- added R34: 10kΩ, PCM_JLCPCB:R_0805, F.Cu at (119.2, 74.0)
- added R35: 10kΩ, PCM_JLCPCB:R_0805, F.Cu at (121.2, 74.0)
- moved J3 0.13 mm to (144.1, 92.1)
Connections:
- U1 pad 41: UART_RTS -> UART_CTS
- U1 pad 42: UART_CTS -> UART_RTS
- U5 pad 13: UART_RTS -> UART_CTS
- U5 pad 5: UART_CTS -> UART_RTS
Routing:
- net BL/BUSY: track 2.05 -> 13.9 mm, vias 0 -> 1
- net UART_TX: track 61.4 -> 65.7 mm
- net VDD: track 38.0 -> 40.9 mm, vias 19 -> 20
- net UART_RX: track 72.9 -> 75.1 mm
- net GND: track 10.0 -> 11.6 mm, vias 137 -> 138
- net UART_RTS: track 20.4 -> 19.5 mm
- net UART_CTS: track 19.5 -> 20.4 mm
Other:
- board size 56.5 x 65 mm -> 56.6 x 65 mm
- board text added: "Orbweaver"
- board text added: "ROM BOOT"
- board text added: "Raspberry Pi Sub-GHz HAT+"
- board text added: "Rev. 1.0"
- board text added: "VESPID"
