File: hardware/orbweaver.kicad_sch (KiCad schematic)
At the start: 40 parts, among them U1 CC1310F128RGZR, Y1 TSX-322524.0000MF15X-AC0, Y2 FC-135_32.7680KA-AG3

Commit message: Fixed firmware python scripts. Updated public schematics.
Parts:
- added J7: DNI, Connector_PinHeader_2.54mm:PinHeader_1x02_P2.54mm_Vertical, symbol Connector:Conn_01x02_Pin
- added R34, R35: 10kΩ, PCM_JLCPCB:R_0805, symbol PCM_JLCPCB-Resistors:0805,10kΩ
Connections:
- net BL/BUSY: now also J7.2 (Pin_2)
- net GND: now also J7.1 (Pin_1)
- net UART_RX: now also R34.2
- net UART_TX: now also R35.2
- net VDD: now also R34.1, R35.1
